File: stigma_core_board/stigma_core_board.kicad_sch (KiCad schematic)
At the start: 93 parts, among them J1 TC2050, J5 USB_C_Receptacle_USB2.0, SW1 KMR721NGLFS, SW2 KMR721NGLFS, U1 STM32H743VITx, U10 H3LIS331DL, U11 MS5607/MS5611, U12 LIS3MDL, U13 BMP580/BMP388/LPS22, U2 TPD4E1U06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

Commit message: Rename LCSC part no. property
Parts:
- C15, C20, C21, C22, C24, C25, C27, C28, C29, C30, C31, C32, C34, C35, C36, C38, C39, C40: LCSC (none) -> C1591; LCSC# C1591 -> (none)
- C18, C23: LCSC (none) -> C14860; LCSC# C14860 -> (none)
- C19: LCSC (none) -> C12891; LCSC# C12891 -> (none)
- C26, C33, C37: LCSC (none) -> C318694; LCSC# C318694 -> (none)
- D4: LCSC (none) -> C167645; LCSC# C167645 -> (none)
- J5: LCSC (none) -> C709357; LCSC# C709357 -> (none)
- R10, R11: LCSC (none) -> C105580; LCSC# C105580 -> (none)
- R12, R13: LCSC (none) -> C107701; LCSC# C107701 -> (none)
- R14, R15, R16, R17, R18, R19, R20, R5, R6: LCSC (none) -> C98220; LCSC# C98220 -> (none)
- SW1, SW2: LCSC (none) -> C2911418; LCSC# C2911418 -> (none)
- U12: LCSC (none) -> C478483; LCSC# C478483 -> (none)
- U4, U6, U9: LCSC (none) -> C784817; LCSC# C784817 -> (none)
- U5: LCSC (none) -> C92102; LCSC# C92102 -> (none)
Changed lines of the file:
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@@
 			)
 		)
-		(property "LCSC#" "C318694"
+		(property "LCSC" "C318694"
 			(at 265.43 142.24 0)
 			(effects
@@
 			)
 		)
-		(property "LCSC#" "C1591"
+		(property "LCSC" "C1591"
 			(at 267.97 33.02 0)
 			(effects
@@
 			)
 		)
-		(property "LCSC#" "C98220"
+		(property "LCSC" "C98220"
 			(at 166.37 201.93 0)
 			(effects
@@
 			)
 		)
-		(property "LCSC#" "C784817"
+		(property "LCSC" "C784817"
 			(at 166.37 52.07 0)
 			(effects
@@
 			)
 		)
-		(property "LCSC#" "C98220"
+		(property "LCSC" "C98220"
 			(at 166.37 222.25 0)
 			(effects
@@
 			)
 		)
-		(property "LCSC#" "C1591"
+		(property "LCSC" "C1591"
 			(at 365.76 209.55 0)
 			(effects
@@
 			)
 		)
-		(property "LCSC#" "C107701"
+		(property "LCSC" "C107701"
 			(at 217.17 245.11 0)
 			(effects
@@
 			)
 		)
-		(property "LCSC#" "C784817"
+		(property "LCSC" "C784817"
 			(at 245.11 190.5 0)
 			(effects
@@
 			)
 		)
-		(property "LCSC#" "C105580"
+		(property "LCSC" "C105580"
 			(at 219.71 231.14 0)
 			(effects
@@
 			)
 		)
-		(property "LCSC#" "C105580"
+		(property "LCSC" "C105580"
 			(at 219.71 233.68 0)
 			(effects
@@
 			)
 		)
-		(property "LCSC#" "C1591"
+		(property "LCSC" "C1591"
 			(at 283.21 190.5 0)
 			(effects
@@
 			)
 		)
-		(property "LCSC#" "C12891"
+		(property "LCSC" "C12891"
 			(at 158.75 257.81 0)
 			(effects
@@
 			)
 		)
-		(property "LCSC#" "C98220"
+		(property "LCSC" "C98220"
 			(at 193.04 237.49 0)
 			(effects
@@
 			)
 		)
-		(property "LCSC#" "C98220"
+		(property "LCSC" "C98220"
 			(at 29.21 54.61 0)
 			(effects
@@
 			)
 		)
-		(property "LCSC#" "C1591"
+		(property "LCSC" "C1591"
 			(at 194.31 52.07 0)
 			(effects
@@
 			)
 		)
-		(property "LCSC#" "C14860"
+		(property "LCSC" "C14860"
 			(at 133.35 257.81 0)
 			(effects
@@
 			)
 		)
-		(property "LCSC#" "C1591"
+		(property "LCSC" "C1591"
 			(at 273.05 190.5 0)
 			(effects
@@
 			)
 		)
-		(property "LCSC#" "C1591"
+		(property "LCSC" "C1591"
 			(at 116.84 240.03 0)
 			(effects
@@
 			)
 		)
-		(property "LCSC#" "C1591"
+		(property "LCSC" "C1591"
 			(at 132.08 214.63 0)
 			(effects
@@
 			)
 		)
-		(property "LCSC#" "C1591"
+		(property "LCSC" "C1591"
 			(at 278.13 33.02 0)
 			(effects
@@
 			)
 		)
-		(property "LCSC#" "C98220"
+		(property "LCSC" "C98220"
 			(at 77.47 218.44 0)
 			(effects
@@
 			)
 		)
-		(property "LCSC#" "C1591"
+		(property "LCSC" "C1591"
 			(at 190.5 93.98 0)
 			(effects
@@
 			)
 		)
-		(property "LCSC#" "C98220"
+		(property "LCSC" "C98220"
 			(at 193.04 229.87 0)
 			(effects
@@
 			)
 		)
-		(property "LCSC#" "C709357"
+		(property "LCSC" "C709357"
 			(at 240.03 241.3 0)
 			(effects
@@
 			)
 		)
-		(property "LCSC#" "C1591"
+		(property "LCSC" "C1591"
 			(at 184.15 125.73 0)
 			(effects
@@
 			)
 		)
-		(property "LCSC#" "C784817"
+		(property "LCSC" "C784817"
 			(at 245.11 142.24 0)
 			(effects
@@
 			)
 		)
-		(property "LCSC#" "C1591"
+		(property "LCSC" "C1591"
 			(at 274.32 142.24 0)
 			(effects
@@
 			)
 		)
-		(property "LCSC#" "C1591"
+		(property "LCSC" "C1591"
 			(at 184.15 52.07 0)
 			(effects
@@
 			)
 		)
-		(property "LCSC#" "C92102"
+		(property "LCSC" "C92102"
 			(at 146.05 252.73 0)
 			(effects
@@
 			)
 		)
-		(property "LCSC#" "C1591"
+		(property "LCSC" "C1591"
 			(at 278.13 80.01 0)
 			(effects
@@
 			)
 		)
-		(property "LCSC#" "C167645"
+		(property "LCSC" "C167645"
 			(at 219.71 226.06 0)
 			(effects
@@
 			)
 		)
-		(property "LCSC#" "C98220"
+		(property "LCSC" "C98220"
 			(at 115.57 226.06 0)
 			(effects
@@
 			)
 		)
-		(property "LCSC#" "C1591"
+		(property "LCSC" "C1591"
 			(at 267.97 80.01 0)
 			(effects
@@
 			)
 		)
-		(property "LCSC#" "C318694"
+		(property "LCSC" "C318694"
 			(at 264.16 190.5 0)
 			(effects
@@
 			)
 		)
-		(property "LCSC#" "C478483"
+		(property "LCSC" "C478483"
 			(at 163.83 163.83 0)
 			(effects
@@
 			)
 		)
-		(property "LCSC#" "C1591"
+		(property "LCSC" "C1591"
 			(at 284.48 142.24 0)
 			(effects
@@
 			)
 		)
-		(property "LCSC#" "C1591"
+		(property "LCSC" "C1591"
 			(at 179.07 166.37 0)
 			(effects
@@
 			)
 		)
-		(property "LCSC#" "C318694"
+		(property "LCSC" "C318694"
 			(at 186.69 156.21 0)
 			(effects
@@
 			)
 		)
-		(property "LCSC#" "C107701"
+		(property "LCSC" "C107701"
 			(at 217.17 240.03 0)
 			(effects
@@
 			)
 		)
-		(property "LCSC#" "C14860"
+		(property "LCSC" "C14860"
 			(at 180.34 93.98 0)
 			(effects
@@
 			)
 		)
-		(property "LCSC#" "C2911418"
+		(property "LCSC" "C2911418"
 			(at 142.24 214.63 0)
 			(effects
@@
 			)
 		)
-		(property "LCSC#" "C98220"
+		(property "LCSC" "C98220"
 			(at 29.21 59.69 0)
 			(effects
@@
 			)
 		)
-		(property "LCSC#" "C1591"
+		(property "LCSC" "C1591"
 			(at 204.47 222.25 0)
 			(effects
@@
 			)
 		)
-		(property "LCSC#" "C98220"
+		(property "LCSC" "C98220"
 			(at 82.55 226.06 0)
 			(effects
@@
 			)
 		)
-		(property "LCSC#" "C1591"
+		(property "LCSC" "C1591"
 			(at 196.85 156.21 0)
 			(effects
@@
 			)
 		)
-		(property "LCSC#" "C2911418"
+		(property "LCSC" "C2911418"
 			(at 166.37 209.55 0)
 			(effects

Commit message: Update LCSC references
Parts:
- C1: LCSC (none) -> C19666
- C10, C9: LCSC (none) -> C12530
- C15, C20, C21, C22, C24, C25, C27, C28, C29, C30, C31, C34, C35, C36, C39, C40: LCSC C1591 -> C1525
- C16, C17, C3, C4, C5, C6, C7: LCSC (none) -> C1525
- C18, C23: LCSC C14860 -> C19702
- C19: LCSC C12891 -> C86295
- C2, C8: LCSC (none) -> C28323
- C26, C33, C37: LCSC C318694 -> C28323
- C32, C38: LCSC C1591 -> C15195
- D1: LCSC (none) -> C2286
- D2: LCSC (none) -> C2296
- D3: LCSC (none) -> C2297
- D4: footprint Diode_SMD:D_SOD-123F -> Diode_SMD:D_SOD-123; LCSC C167645 -> C8598
- FB1: LCSC (none) -> C1002
- J3: now not fitted
- R1, R2, R3, R4: LCSC (none) -> C17168
- R10, R11: LCSC C105580 -> C25905
- R12, R13: LCSC C107701 -> C25092
- R14: LCSC C98220 -> C25900
- R15: LCSC C98220 -> C25744
- R16, R17, R18, R19, R20: LCSC C98220 -> C25092
- R5: LCSC C98220 -> C25741
- R6: LCSC C98220 -> C11702
- R7, R8, R9: LCSC (none) -> C11702
- U1: LCSC (none) -> C730183
- U10: LCSC (none) -> C2655074
- U11: LCSC (none) -> C97627
- U13: value BMP580/BMP388/LPS22 -> BMP580; LCSC (none) -> C22391138
- U2, U7: LCSC (none) -> C527516
- U3: value BMP580/BMP388/LPS22 -> LPS22; LCSC (none) -> C2827824
- U4: LCSC C784817 -> C2988404
- U6: value ICM-42688 (or other LGA-14 IMU) -> ICM-42688-P; LCSC C784817 -> C1850418
- U8: LCSC (none) -> C190862
- Y1: LCSC (none) -> C9006
- Y2: LCSC (none) -> C70509

Commit message: Minor layout tweaks
Other:
- note removed: "TODO: additional input capacitance?"
- note removed: "TODO: button footprint?"
- note removed: "TODO: replace with BMP585, ICP 20100? Another LGA-10 footprint?"
Changed lines of the file:
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@@
 		)
 	)
-	(text "TODO: replace with BMP585, ICP 20100? Another LGA-10 footprint?"
-		(exclude_from_sim no)
-		(at 291.084 90.17 90)
-		(effects
-			(font
-				(size 1.27 1.27)
-			)
-		)
-	)
-	(text "TODO: additional input capacitance?"
-		(exclude_from_sim no)
-		(at 355.092 162.306 0)
-		(effects
-			(font
-				(size 1.27 1.27)
-			)
-		)
-	)
-	(text "TODO: button footprint?"
-		(exclude_from_sim no)
-		(at 143.51 194.056 0)
-		(effects
-			(font
-				(size 1.27 1.27)
-			)
-		)
-	)
 	(text "Of the two USB peripherals, we use\nthis one, because PA11/PA12 are what\nthe bootloader uses for DFU."
 		(exclude_from_sim no)
@@
 			)
 		)
-		(property "Description" "TODO: LCSC"
+		(property "Description" ""
 			(at 240.03 241.3 0)
 			(effects
