File: stigma_core_board/stigma_core_board.kicad_sch (KiCad schematic)
At the start: 93 parts, among them J1 TC2050, J3 CONN PLUG 70POS SMD GOLD, J5 USB_C_Receptacle_USB2.0, SW1 KMR721NGLFS, SW2 KMR721NGLFS, U1 STM32H743VIT6, U10 H3LIS331DL, U11 MS5607/MS5611, U12 LIS3MDL, U13 BMP580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

Commit message: core: Final bom changes, production files
Parts:
- C2, C26, C33, C37, C8: LCSC C28323 -> C52923
- D2: LCSC C2296 -> C72038
- D3: LCSC C2297 -> C965804
- J3: now in the parts list
- R12, R13: value 22R -> 22
Changed lines of the file:
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@@
 			)
 		)
-		(property "LCSC" "C28323"
+		(property "LCSC" "C52923"
 			(at 265.43 142.24 0)
 			(effects
@@
 			)
 		)
-		(property "LCSC" "C28323"
+		(property "LCSC" "C52923"
 			(at 86.36 27.94 0)
 			(effects
@@
 			)
 		)
-		(property "Value" "22R"
+		(property "Value" "22"
 			(at 218.948 246.888 90)
 			(effects
@@
 		(unit 1)
 		(exclude_from_sim no)
-		(in_bom no)
+		(in_bom yes)
 		(on_board yes)
 		(dnp no)
@@
 			)
 		)
-		(property "Description" "populated manually"
+		(property "Description" ""
 			(at 356.87 101.6 0)
 			(effects
@@
 			)
 		)
-		(property "LCSC" "C28323"
+		(property "LCSC" "C52923"
 			(at 264.16 190.5 0)
 			(effects
@@
 			)
 		)
-		(property "LCSC" "C28323"
+		(property "LCSC" "C52923"
 			(at 102.87 27.94 0)
 			(effects
@@
 			)
 		)
-		(property "LCSC" "C2297"
+		(property "LCSC" "C965804"
 			(at 39.37 274.32 0)
 			(effects
@@
 			)
 		)
-		(property "LCSC" "C28323"
+		(property "LCSC" "C52923"
 			(at 186.69 156.21 0)
 			(effects
@@
 			)
 		)
-		(property "Value" "22R"
+		(property "Value" "22"
 			(at 217.424 242.062 90)
 			(effects
@@
 			)
 		)
-		(property "LCSC" "C2296"
+		(property "LCSC" "C72038"
 			(at 39.37 265.43 0)
 			(effects
