File: stigma_mission_board_hyacinth/voltage_regulator.kicad_sch (KiCad schematic)
At the start: 19 parts, among them U15 TPS62933

Commit message: added some comments
Parts:
- L1: Würth Nr: (none) -> 74439346068(?)
Other:
- note added: "@todo: check inductor"
- note added: "@todo: use 0402 resistor to decrease loop"
- note added: "@todo: use high quality capacitors with sufficient voltage rating"

Commit message: improve can traces at VB, use smaller resistor for voltage reg.
Parts:
- R68: footprint Resistor_SMD:R_0603_1608Metric -> Resistor_SMD:R_0402_1005Metric
- U15: Example Layout www.ti.com/lit/ds/symlink/tps62933.pdf -> https://www.ti.com/lit/ug/sluuch1/sluuch1.pdf
Changed lines of the file:
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@@
 			)
 		)
-		(property "Footprint" "Resistor_SMD:R_0603_1608Metric"
+		(property "Footprint" "Resistor_SMD:R_0402_1005Metric"
 			(at 156.21 93.218 90)
 			(effects
@@
 			)
 		)
-		(property "Example Layout" "www.ti.com/lit/ds/symlink/tps62933.pdf"
+		(property "Example Layout" "https://www.ti.com/lit/ug/sluuch1/sluuch1.pdf"
 			(at 139.7 99.06 0)
 			(effects

Commit message: design check finished, some cosmetic changes, part adaptions, prints, etc.
Parts:
- C53: LCSC (none) -> C7419416
- C55, C56: LCSC (none) -> C45783
- C57: LCSC (none) -> C1525
- R68: LCSC # C21189 -> C106231
Other:
- note removed: "@todo: Diode können wir weglassen oder?"
- note removed: "@todo: check inductor"
- note removed: "@todo: use 0402 resistor to decrease loop"
Changed lines of the file:
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@@
 	(generator_version "9.0")
 	(paper "A4")
-	(text "@todo: Diode können wir weglassen oder?"
-		(exclude_from_sim no)
-		(at 213.106 83.312 0)
-		(effects
-			(font
-				(size 1.27 1.27)
-			)
-		)
-	)
 	(text "Enable input to the converter.\nDriving EN high or leaving this\npin floating enable the converter.\n(Datasheet page 3)"
 		(exclude_from_sim no)
@@
 		)
 	)
-	(text "@todo: check inductor"
-		(exclude_from_sim no)
-		(at 179.324 86.868 0)
-		(effects
-			(font
-				(size 1.27 1.27)
-			)
-		)
-	)
-	(text "@todo: use 0402 resistor to decrease loop"
-		(exclude_from_sim no)
-		(at 162.56 96.52 0)
-		(effects
-			(font
-				(size 1.27 1.27)
-			)
-		)
-	)
 	(text "@todo: use high quality capacitors with sufficient voltage rating"
 		(exclude_from_sim no)
@@
 			)
 		)
+		(property "LCSC" "C1525"
+			(at 208.28 95.25 0)
+			(effects
+				(font
+					(size 1.27 1.27)
+				)
+				(hide yes)
+			)
+		)
 		(pin "2"
 		)
@@
 			)
 		)
+		(property "LCSC" "C45783"
+			(at 189.23 95.25 0)
+			(effects
+				(font
+					(size 1.27 1.27)
+				)
+				(hide yes)
+			)
+		)
 		(pin "2"
 		)
@@
 			)
 		)
+		(property "LCSC" "C7419416"
+			(at 123.19 109.22 0)
+			(effects
+				(font
+					(size 1.27 1.27)
+				)
+				(hide yes)
+			)
+		)
 		(pin "2"
 		)
@@
 			)
 		)
-		(property "LCSC #" "C21189"
+		(property "LCSC #" "C106231"
 			(at 156.21 91.44 90)
 			(effects
@@
 			(at 199.39 95.25 0)
 			(effects
+				(font
+					(size 1.27 1.27)
+				)
+				(hide yes)
+			)
+		)
+		(property "LCSC" "C45783"
+			(at 199.39 95.25 0)
+			(effects

Commit message: finished req. checklist, marginal changes
Parts:
- L1: now not fitted
Changed lines of the file:
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@@
 		(in_bom yes)
 		(on_board yes)
-		(dnp no)
+		(dnp yes)
 		(property "Reference" "L1"
 			(at 180.34 89.408 90)

Commit message: some lcsc number changes
Parts:
- C24, C6: LCSC (none) -> C19702; LCSC# C96446 -> (none)
- C52: LCSC# C1525 -> C1525
- C54: LCSC (none) -> C1525
- C55, C56: LCSC C45783 -> C59461
- R67: LCSC (none) -> C21189; LCSC# C21189 -> (none)
- R68: LCSC (none) -> C17168; LCSC # C106231 -> (none)
- R70: LCSC (none) -> C25804; LCSC# C25804 -> (none)
Changed lines of the file:
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@@
 			)
 		)
-		(property "LCSC#" "C25804 "
+		(property "LCSC" "C25804 "
 			(at 156.21 114.3 0)
 			(effects
@@
 					(size 1.27 1.27)
 				)
-				(hide yes)
 			)
 		)
@@
 			)
 		)
-		(property "LCSC" "C45783"
+		(property "LCSC" "C59461"
 			(at 189.23 95.25 0)
 			(effects
@@
 			)
 		)
+		(property "LCSC" " C1525"
+			(at 167.64 91.44 90)
+			(effects
+				(font
+					(size 1.27 1.27)
+				)
+				(hide yes)
+			)
+		)
 		(pin "2"
 		)
@@
 			)
 		)
-		(property "LCSC #" "C106231"
+		(property "LCSC" "C17168"
 			(at 156.21 91.44 90)
 			(effects
@@
 					(size 1.27 1.27)
 				)
-				(hide yes)
 			)
 		)
@@
 			)
 		)
-		(property "LCSC#" "C1525"
+		(property "LCSC#" " C1525"
 			(at 86.36 95.25 0)
 			(effects
@@
 			)
 		)
-		(property "LCSC#" "C96446"
+		(property "LCSC" "C19702"
 			(at 74.93 95.25 0)
 			(effects
@@
 			)
 		)
-		(property "LCSC" "C45783"
+		(property "LCSC" "C59461"
 			(at 199.39 95.25 0)
 			(effects
@@
 			)
 		)
-		(property "LCSC#" "C96446"
+		(property "LCSC" "C19702"
 			(at 63.5 95.25 0)
 			(effects
@@
 			)
 		)
-		(property "LCSC#" "C21189"
+		(property "LCSC" "C21189"
 			(at 129.54 133.35 0)
 			(effects
